File: amoeba/amoeba.sch (KiCad schematic (older format))
At the start: 14 parts

Commit message: Cleaned up Amoeba PCB.
Parts:
- removed D1: DIODE, ~, symbol DIODE
- removed LC0, LC1, LC2, LR0, LR1, SC0, SC1, SC2, SR0, SR1: CONN_1, symbol CONN_1
- removed LED1: LED, ~, symbol LED
- removed R1: RESISTOR, ~, symbol RESISTOR
- removed S1: MX1A, ~, symbol MX1A
- added LC0:0, LC0:1, LC0:2, LR0:0, LR0:1, SC0:0, SC0:1, SC0:2, SR0:0, SR0:1: CONN_1, symbol CONN_1
Connections:
- new net key/LC0: LC0:0.1
- new net key/LC1: LC0:1.1, LC0:2.1
- new net key/LR0: LR0:0.1
- new net key/LR1: LR0:1.1
- new net key/SC0: SC0:0.1
- new net key/SC1: SC0:1.1, SC0:2.1
- new net key/SR0: SR0:0.1
- new net key/SR1: SR0:1.1
Other:
- note removed: "In-switch LED"
- note removed: "LED row"
- note removed: "LED\ncolumn"
- note removed: "LED\nresistor"
- note removed: "Switch row"
- note removed: "Switch\n"
- note removed: "Switch\ncolumn"
- note removed: "Switch\ndiode"
