File: amoeba-stabilizer-2/amoeba-stabilizer-2.kicad_pcb (KiCad board)
At the start: 2 copper layers, 35.1 x 20.8 mm, 42 parts

Commit message: Update to version 1.5.
Parts:
- removed amoeba-round-cu: G***, amoeba-round-cu
- added amoeba-round: G***, amoeba-round, F.Cu at (238.0, 110.9)
Other:
- board text added: "v1.5"
- board text removed: "v1.3"
