File: amoeba-king/amoeba-royale.kicad_pcb (KiCad board)
At the start: 2 copper layers, 19.1 x 19.1 mm, 7 parts, among them J1 Conn_01x05_Male, J2 Conn_01x05_Male, J3 Conn_01x05_Male, J4 Conn_01x05_Male

Commit message: Getting closer
3d View still has pins :(
Parts:
- D1: value DIODE -> 1N4148W-7-F; footprint Diode_SMD:D_0805_2012Metric_Pad1.15x1.40mm_HandSolder -> Diode_SMD:D_SOD-323
- J1, J2, J4: footprint Connector_PinHeader_1.27mm:PinHeader_1x05_P1.27mm_Vertical -> amoeba-modules:Header_1x05_P1.27mm; moved to B.Cu
- J3: value Conn_01x05_Male -> Conn_01x04_Male; footprint Connector_PinHeader_1.27mm:PinHeader_1x05_P1.27mm_Vertical -> amoeba-modules:Header_1x04_P1.27mm; moved to B.Cu
- LED1: value SK6812MINI -> SK6812MINI_E
- moved D1 0.38 mm to (133.9, 124.7), turned to 0 degrees
- turned J1 to 270 degrees
- turned J2 to 180 degrees
- turned J3 to 270 degrees
- turned J4 to 180 degrees
Connections:
- D1 pad 1: Net-(D1-Pad1) -> /C
- D1 pad 2: /C -> Net-(D1-Pad2)
- LED1 pad 1: /DOUT -> /VDD
- LED1 pad 2: /GND -> /DOUT
- LED1 pad 3: /DIN -> /GND
- LED1 pad 4: /VDD -> /DIN
- S1 pad 2: Net-(D1-Pad1) -> Net-(D1-Pad2)
Routing:
- net Net-(D1-Pad2): track 0.00 -> 4.66 mm
- net /GND: track 18.6 -> 14.1 mm, vias 15 -> 18
- net Net-(D1-Pad1): track 3.85 -> 0.00 mm
- net /VDD: track 34.2 -> 36.2 mm
- net /C: track 18.4 -> 16.6 mm, vias 2 -> 0
- net /DOUT: track 29.8 -> 31.2 mm, vias 2 -> 1
- net /DIN: track 33.2 -> 32.5 mm

Commit message: Getting ready for final review, before sending for production
Parts:
- added J5: Conn_01x01_Male, amoeba-modules:Header_1x01_P1.27mm, B.Cu at (80.5, 176.1)
- added J6: Conn_01x01_Male, amoeba-modules:Header_1x01_P1.27mm, B.Cu at (80.4, 161.2)
- moved D1 80.1 mm to (68.5, 171.0), turned to 180 degrees
- moved J1 79.9 mm to (73.0, 176.1), turned to 90 degrees
- moved J2 76.1 mm to (67.9, 166.2), turned to 0 degrees
- moved S1 66.3 mm to (75.4, 168.7), turned to 0 degrees
- moved J3 62.4 mm to (73.0, 161.2), turned to 90 degrees
- moved LED1 60.4 mm to (75.4, 163.6), turned to 180 degrees
- moved J4 51.9 mm to (82.9, 166.2), turned to 0 degrees
Routing:
- net /C: track 16.6 -> 38.4 mm
- net /GND: vias 18 -> 20
Other:
- board size 19.1 x 19.1 mm -> 19 x 19.1 mm
- board text added: "C"
- board text added: "DI"
- board text added: "DO"
- board text added: "G"
- board text added: "R"
- board text added: "V"
