File: amoeba-king/amoeba-royale.sch (KiCad schematic (older format))
At the start: 4 parts, among them J1 Conn_01x05_Male, J2 Conn_01x05_Male, J3 Conn_01x05_Male, J4 Conn_01x05_Male

Commit message: Getting closer
3d View still has pins :(
Parts:
- removed J3: Conn_01x05_Male, Connector_PinHeader_1.27mm:PinHeader_1x05_P1.27mm_Vertical, symbol Connector:Conn_01x05_Male
- added J3: Conn_01x04_Male, amoeba-modules:Header_1x04_P1.27mm, symbol Connector:Conn_01x04_Male
- J1, J2, J4: footprint Connector_PinHeader_1.27mm:PinHeader_1x05_P1.27mm_Vertical -> amoeba-modules:Header_1x05_P1.27mm
Connections:
- net C: now also J3.3 (Pin_3)
- net DOUT: now also J3.1 (Pin_1)
- net GND: now also J3.4 (Pin_4)
- net VDD: now also J3.2 (Pin_2)
Changed lines of the file:
@@
 F 0 "J2" H 6472 3224 50  0000 R CNN
 F 1 "Conn_01x05_Male" H 6472 3133 50  0000 R CNN
-F 2 "Connector_PinHeader_1.27mm:PinHeader_1x05_P1.27mm_Vertical" H 6500 3200 50  0001 C CNN
+F 2 "amoeba-modules:Header_1x05_P1.27mm" H 6500 3200 50  0001 C CNN
 F 3 "~" H 6500 3200 50  0001 C CNN
 	1    6500 3200
@@
 F 0 "J4" H 4150 3600 50  0000 C CNN
 F 1 "Conn_01x05_Male" H 4200 2950 50  0000 C CNN
-F 2 "Connector_PinHeader_1.27mm:PinHeader_1x05_P1.27mm_Vertical" H 4200 3250 50  0001 C CNN
+F 2 "amoeba-modules:Header_1x05_P1.27mm" H 4200 3250 50  0001 C CNN
 F 3 "~" H 4200 3250 50  0001 C CNN
 	1    4200 3250
@@
 F 0 "J1" V 5462 1912 50  0000 R CNN
 F 1 "Conn_01x05_Male" V 5553 1912 50  0000 R CNN
-F 2 "Connector_PinHeader_1.27mm:PinHeader_1x05_P1.27mm_Vertical" H 5400 2200 50  0001 C CNN
+F 2 "amoeba-modules:Header_1x05_P1.27mm" H 5400 2200 50  0001 C CNN
 F 3 "~" H 5400 2200 50  0001 C CNN
 	1    5400 2200
@@
 Text Label 4450 3150 0    50   ~ 0
 VDD
+$Comp
+L Connector:Conn_01x04_Male J3
+U 1 1 5EC2A986
+P 5250 4400
+F 0 "J3" V 5404 4112 50  0000 R CNN
+F 1 "Conn_01x04_Male" V 5313 4112 50  0000 R CNN
+F 2 "amoeba-modules:Header_1x04_P1.27mm" H 5250 4400 50  0001 C CNN
+F 3 "~" H 5250 4400 50  0001 C CNN
+	1    5250 4400
+	0    -1   -1   0
+$EndComp
 Wire Bus Line
 	6050 2600 6050 3950
@@
 Wire Bus Line
 	4650 2600 4650 3950
-$Comp
-L Connector:Conn_01x05_Male J3
-U 1 1 5EC34669
-P 5350 4400
-F 0 "J3" V 5504 4112 50  0000 R CNN
-F 1 "Conn_01x05_Male" V 5413 4112 50  0000 R CNN
-F 2 "Connector_PinHeader_1.27mm:PinHeader_1x05_P1.27mm_Vertical" H 5350 4400 50  0001 C CNN
-F 3 "~" H 5350 4400 50  0001 C CNN
-	1    5350 4400
-	0    -1   -1   0
-$EndComp
 $EndSCHEMATC

Commit message: Getting ready for final review, before sending for production
Parts:
- added J5, J6: Conn_01x01_Male, amoeba-modules:Header_1x01_P1.27mm, symbol Connector:Conn_01x01_Male
Connections:
- net C: now also J5.1 (Pin_1), J6.1 (Pin_1)
Changed lines of the file:
@@
 	0    -1   -1   0
 $EndComp
+$Comp
+L Connector:Conn_01x01_Male J5
+U 1 1 5EC458E5
+P 4800 2200
+F 0 "J5" V 4862 2244 50  0000 L CNN
+F 1 "Conn_01x01_Male" V 4953 2244 50  0000 L CNN
+F 2 "amoeba-modules:Header_1x01_P1.27mm" H 4800 2200 50  0001 C CNN
+F 3 "~" H 4800 2200 50  0001 C CNN
+	1    4800 2200
+	0    1    1    0
+$EndComp
+$Comp
+L Connector:Conn_01x01_Male J6
+U 1 1 5EC464E7
+P 4750 4400
+F 0 "J6" V 4904 4312 50  0000 R CNN
+F 1 "Conn_01x01_Male" V 4813 4312 50  0000 R CNN
+F 2 "amoeba-modules:Header_1x01_P1.27mm" H 4750 4400 50  0001 C CNN
+F 3 "~" H 4750 4400 50  0001 C CNN
+	1    4750 4400
+	0    -1   -1   0
+$EndComp
+Entry Wire Line
+	4750 4050 4850 3950
+Entry Wire Line
+	4700 2600 4800 2500
+Wire Wire Line
+	4800 2500 4800 2400
+Wire Wire Line
+	4750 4200 4750 4050
+Text Label 4800 2500 1    50   ~ 0
+C
+Text Label 4750 4200 1    50   ~ 0
+C
 Wire Bus Line
 	6050 2600 6050 3950
