File: amoeba-king/amoeba-king.kicad_pcb (KiCad board)
At the start: 2 copper layers, 19 x 19.1 mm, 14 parts, among them J1 Conn_01x04_Male, J2 Conn_01x04_Male, J3 Conn_01x04_Male, J4 Conn_01x04_Male, J5 Conn_01x01_Male, J6 Conn_01x01_Male

Commit message: Cleanup tracks.
Routing:
- net /DIN: track 5.74 -> 4.65 mm
- net /DOUT: track 3.26 -> 2.72 mm
Changed lines of the file:
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@@
   (via (at 78.9432 166.878) (size 0.6) (drill 0.4) (layers "F.Cu" "B.Cu") (net 1))
   (via (at 78.7855 162.8394) (size 0.6) (drill 0.4) (layers "F.Cu" "B.Cu") (net 1))
-  (segment (start 79.1464 167.0812) (end 78.9432 166.878) (width 0.254) (layer "B.Cu") (net 1))
-  (segment (start 78.7855 162.8394) (end 78.7721 162.826) (width 0.254) (layer "B.Cu") (net 1))
-  (segment (start 78.7721 162.826) (end 77.988 162.826) (width 0.254) (layer "B.Cu") (net 1))
   (segment (start 80.747222 163.733078) (end 80.2132 164.2671) (width 0.254) (layer "F.Cu") (net 2))
   (segment (start 76.252441 166.116) (end 74.3966 166.116) (width 0.254) (layer "F.Cu") (net 2))
@@
   (via (at 80.747222 163.733078) (size 0.6) (drill 0.4) (layers "F.Cu" "B.Cu") (net 2))
   (via (at 73.1012 166.878) (size 0.6) (drill 0.4) (layers "F.Cu" "B.Cu") (net 2))
-  (segment (start 80.2232 166.878) (end 80.2132 166.878) (width 0.254) (layer "B.Cu") (net 2))
   (segment (start 80.7773 163.703) (end 82.9056 163.703) (width 0.254) (layer "B.Cu") (net 2))
-  (segment (start 80.747222 163.733078) (end 80.7773 163.703) (width 0.254) (layer "B.Cu") (net 2))
   (segment (start 72.3392 164.338) (end 71.9474 164.7298) (width 0.254) (layer "F.Cu") (net 3))
   (segment (start 71.9474 164.7298) (end 71.9474 166.878) (width 0.254) (layer "F.Cu") (net 3))
@@
   (via (at 72.3392 164.338) (size 0.6) (drill 0.4) (layers "F.Cu" "B.Cu") (net 3))
   (segment (start 72.876 164.338) (end 72.888 164.326) (width 0.254) (layer "B.Cu") (net 3))
-  (segment (start 72.3392 164.338) (end 72.876 164.338) (width 0.254) (layer "B.Cu") (net 3))
   (segment (start 71.6788 161.282) (end 72.03129 161.63449) (width 0.254) (layer "B.Cu") (net 4))
   (segment (start 71.6788 161.281294) (end 71.6788 160.782) (width 0.254) (layer "B.Cu") (net 4))
@@
   (via (at 78.9178 165.608) (size 0.6) (drill 0.4) (layers "F.Cu" "B.Cu") (net 11))
   (segment (start 71.9474 165.598) (end 71.9828 165.6334) (width 0.254) (layer "B.Cu") (net 11))
-  (segment (start 78.9278 165.598) (end 78.9432 165.598) (width 0.254) (layer "B.Cu") (net 11))
-  (segment (start 78.8924 165.6334) (end 78.9178 165.608) (width 0.254) (layer "B.Cu") (net 11))
   (segment (start 71.9828 165.6334) (end 78.8924 165.6334) (width 0.254) (layer "B.Cu") (net 11))
-  (segment (start 78.9178 165.608) (end 78.9278 165.598) (width 0.254) (layer "B.Cu") (net 11))
   (zone (net 5) (net_name "/GND") (layer "F.Cu") (hatch edge 0.508)
     (connect_pads (clearance 0.1))
